File: uCBoardBase/uCBoardBase.brd (EAGLE design)
At the start: 85.1 x 70.8 mm, 49 parts, among them J1 POWER_JACKPTH, U1 TM4C123BE6PMSMD, U2 TPS73633DBVR, U4 FT230XSSOP, Y1 16 MHz, Y2 32.768 kHz

Commit message: Updated README
Parts:
- added CC_TEXT1, CC_TEXT2: CREATIVE_COMMONS, SparkFun-Aesthetics:CREATIVE_COMMONS
Other:
- board text added: "B. Carrizales"
Changed lines of the file:
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@@
 <text x="43.815" y="68.58" size="1.27" layer="21" rot="R270">GND</text>
 <text x="41.275" y="68.58" size="1.27" layer="21" rot="R270">VBAT</text>
+<text x="60.96" y="-6.35" size="1.778" layer="51" rot="R180">B. Carrizales</text>
 </plain>
 <attributes>
@@
 <element name="LED4" library="SparkFun-LED" package="LED-0603" value="" x="34.29" y="52.07" rot="R180"/>
 <element name="R9" library="SparkFun-Passives" package="0603-RES" value="0" x="38.1" y="53.34" rot="R180"/>
+<element name="CC_TEXT1" library="SparkFun-Aesthetics" package="CREATIVE_COMMONS" value="CREATIVE_COMMONS" x="20.32" y="-7.62"/>
+<element name="CC_TEXT2" library="SparkFun-Aesthetics" package="CREATIVE_COMMONS" value="CREATIVE_COMMONS" x="20.32" y="-7.62"/>
 </elements>
 <signals>
